Commit message: unfinished code

File: simulation/Hand-Assem-By-Part-URDF.SLDASM/urdf/Example Sphere.urdf (robot description, URDF)
Before this commit: robot Example Sphere, 1 links, 0 joints
Links:
- link Example Sphere: geometry collision mesh filename=package://Hand-Assem-By-Part-URDF.SLDASM/meshes/Example Sph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; visual mesh filename=package://Hand-Assem-By-Part-URDF.SLDASM/meshes/Example Sph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
